File: Monopolyzaehler2.0/Tiefenentladeschutz-addon.brd (EAGLE design)
At the start: 51.2 x 38 mm, 10 parts, among them IC1 ICL7665CSA, X1 MKDSN1,5/2-5,08

Commit message: Addon für Tiefenentladeschutz LiPo
Routing:
- net V+: track 63.1 -> 66.9 mm
Other:
- board text added: "+"
- board text added: "-"
- board text added: "9-6V"
- board text added: "LiPo Adapter v1.1 02/2016"
- board text added: "Monopoly LiPo Adapter mit Tiefenentladeschutz bei 6.2V V 1.1 02/2017"
Changed lines of the file:
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@@
 <wire x1="51" y1="6.4" x2="51" y2="38" width="0.4064" layer="20"/>
 <circle x="47.2" y="10" radius="0.925" width="1.551" layer="116"/>
+<text x="40" y="32.4" size="3.81" layer="1" font="vector">+</text>
+<text x="43.2" y="28" size="3.81" layer="1" font="vector" rot="R90">-</text>
+<text x="49.8" y="13.4" size="1.6764" layer="1" font="vector" ratio="12" rot="R90">LiPo Adapter
+v1.1 02/2016</text>
+<text x="44.4" y="10.6" size="1.4224" layer="1" font="vector" ratio="12" rot="R180">9-6V</text>
+<text x="-11.4" y="45" size="1.778" layer="1">Monopoly LiPo Adapter
+mit Tiefenentladeschutz bei 6.2V
+V 1.1  02/2017</text>
 </plain>
 <attributes>
@@
 <wire x1="42.2" y1="12.6" x2="42.2" y2="13.578" width="0.4064" layer="1"/>
 <wire x1="42.2" y1="13.578" x2="42.3" y2="13.678" width="0.4064" layer="1"/>
-<wire x1="35.375" y1="34.3189" x2="42.4811" y2="34.3189" width="0.4064" layer="1"/>
-<wire x1="42.4811" y1="34.3189" x2="44" y2="32.8" width="0.4064" layer="1"/>
-<wire x1="44" y1="32.8" x2="44" y2="14" width="0.4064" layer="1"/>
+<wire x1="44" y1="35.2" x2="44" y2="14" width="0.4064" layer="1"/>
 <wire x1="44" y1="14" x2="43.8" y2="13.8" width="0.4064" layer="1"/>
 <wire x1="43.8" y1="13.8" x2="42.422" y2="13.8" width="0.4064" layer="1"/>
@@
 <wire x1="27.54" y1="16.55" x2="28.95" y2="16.55" width="0.4064" layer="1"/>
 <wire x1="28.95" y1="16.55" x2="31" y2="18" width="0.4064" layer="1"/>
+<wire x1="35.375" y1="34.3189" x2="35.375" y2="34.975" width="0.4064" layer="1"/>
+<wire x1="35.375" y1="34.975" x2="37.2" y2="36.8" width="0.4064" layer="1"/>
+<wire x1="37.2" y1="36.8" x2="42.4" y2="36.8" width="0.4064" layer="1"/>
+<wire x1="42.4" y1="36.8" x2="44" y2="35.2" width="0.4064" layer="1"/>
 </signal>
 <signal name="N$13">
@@
 </board>
 </drawing>
+<compatibility>
+<note version="6.3" minversion="6.2.2" severity="warning">
+Since Version 6.2.2 text objects can contain more than one line,
+which will not be processed correctly with this version.
+</note>
+</compatibility>
 </eagle>
